File: HB-SEN-BME280_EXP625.kicad_sch (KiCad schematic)
At the start: 23 parts, among them J2 ISP, J3 FTDI, Q1 IRLU024N, SW1 CONFIG, SW2 RESET, U1 Arduino_Pro_Mini_328P, U2 CC1101, U3 BME280

Commit message: :bug: Fix resistor value in voltage divider
Parts:
- BT1, BT2: value (none) -> AA; footprint (none) -> HB-SEN-BME280_EXP625:BatterHolder_6S-AA
- R6: value 47k -> (none)
Changed lines of the file:
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@@
       (effects (font (size 1.27 1.27)) (justify left))
     )
-    (property "Value" "" (id 1) (at 33.02 39.8779 0)
-      (effects (font (size 1.27 1.27)) (justify left))
-    )
-    (property "Footprint" "" (id 2) (at 29.21 39.116 90)
+    (property "Value" "AA" (id 1) (at 33.02 39.8779 0)
+      (effects (font (size 1.27 1.27)) (justify left))
+    )
+    (property "Footprint" "HB-SEN-BME280_EXP625:BatterHolder_6S-AA" (id 2) (at 29.21 39.116 90)
       (effects (font (size 1.27 1.27)) hide)
     )
@@
       (effects (font (size 1.27 1.27)) (justify left))
     )
-    (property "Value" "" (id 1) (at 49.53 39.8779 0)
-      (effects (font (size 1.27 1.27)) (justify left))
-    )
-    (property "Footprint" "" (id 2) (at 39.37 41.91 90)
+    (property "Value" "AA" (id 1) (at 49.53 39.8779 0)
+      (effects (font (size 1.27 1.27)) (justify left))
+    )
+    (property "Footprint" "HB-SEN-BME280_EXP625:BatterHolder_6S-AA" (id 2) (at 39.37 41.91 90)
       (effects (font (size 1.27 1.27)) hide)
     )
@@
     (in_bom yes) (on_board yes)
     (property "Reference" "R6" (id 0) (at 236.22 129.54 90))
-    (property "Value" "47k" (id 1) (at 236.22 132.08 90))
+    (property "Value" "" (id 1) (at 236.22 132.08 90))
     (property "Footprint" "Resistor_THT:R_Axial_DIN0207_L6.3mm_D2.5mm_P2.54mm_Vertical" (id 2) (at 236.22 133.858 90)
       (effects (font (size 1.27 1.27)) hide)
@@
     )
     (path "/eb8be287-6c70-4326-b689-dbfac252f7ab"
-      (reference "R6") (unit 1) (value "47k") (footprint "Resistor_THT:R_Axial_DIN0207_L6.3mm_D2.5mm_P2.54mm_Vertical")
+      (reference "R6") (unit 1) (value "220k") (footprint "Resistor_THT:R_Axial_DIN0207_L6.3mm_D2.5mm_P2.54mm_Vertical")
     )
     (path "/6ad65c37-7515-4fb3-aaf8-1a0633093c90"
